Commit message: clean up xacro

File: kuka_lbr_iisy_support/urdf/lbr_iisy11_r1300_macro.xacro (robot description, xacro)
@@ -5,10 +5,7 @@
   <xacro:include filename="$(find kuka_resources)/urdf/common_materials.xacro"/>
   <xacro:include filename="$(find kuka_lbr_iisy_support)/urdf/lbr_iisy_transmission.xacro"/>
-  <xacro:macro name="kuka_lbr_iisy11_r1300_robot" params="prefix controller_ip client_ip use_fake_hardware qos_config_file *origin">
-    <!-- ros2 control instance -->
-    <xacro:kuka_lbr_iisy_ros2_control name="${prefix}lbr_iisy11_r1300" prefix="${prefix}" client_ip="${client_ip}" controller_ip="${controller_ip}" use_fake_hardware="${use_fake_hardware}" qos_config_file="${qos_config_file}"/>
+  <xacro:macro name="kuka_lbr_iisy11_r1300_robot" params="prefix">
     <!-- links - main serial chain -->
-    <link name="world"/>
-    <link name="${prefix}base_link">
+     <link name="${prefix}base_link">
       <collision>
         <geometry>
@@ -151,9 +148,9 @@
     </link>
     <!-- joints - main serial chain -->
-    <joint name="${prefix}world-base_link" type="fixed">
+<!--    <joint name="${prefix}world-base_link" type="fixed">
       <parent link="world"/>
       <child link="${prefix}base_link"/>
       <xacro:insert_block name="origin"/>
-    </joint>
+    </joint>-->
     <joint name="${prefix}joint_1" type="revolute">
       <axis xyz="0.0 0.0 1.0"/>
